Commit message: plugin works

File: robot/urdf/main_urdf.URDF (robot description, URDF)
Before this commit: robot zahlil, 5 links, 4 joints
Links:
- link back_left_link: geometry collision cylinder length=0.02 radius=0.078; collision cylinder length=0.02 radius=0.078
- link back_right_link: geometry collision cylinder length=0.02 radius=0.078; collision cylinder length=0.02 radius=0.078
- link front_left_link: geometry collision cylinder length=0.02 radius=0.078; collision cylinder length=0.02 radius=0.078
- link front_right_link: geometry collision cylinder length=0.02 radius=0.078; collision cylinder length=0.02 radius=0.078

Commit message: or

File: robot/urdf/main_urdf.URDF (robot description, URDF)
Before this commit: robot zahlil, 5 links, 4 joints
Links:
- link back_left_link: geometry collision cylinder length=0.02 radius=0.08; collision cylinder length=0.02 radius=0.08
- link back_right_link: geometry collision cylinder length=0.02 radius=0.08; collision cylinder length=0.02 radius=0.08
- link front_left_link: geometry collision cylinder length=0.02 radius=0.08; collision cylinder length=0.02 radius=0.08
- link front_right_link: geometry collision cylinder length=0.02 radius=0.08; collision cylinder length=0.02 radius=0.08
